Commit message: Rename package appropriately

File: self_localizing_robot/urdf/rover.xacro (robot description, xacro)
@@ -1,6 +1,6 @@
 <?xml version='1.0'?>
-<robot name="my_robot" xmlns:xacro="http://www.ros.org/wiki/xacro">
-  <xacro:include filename="$(find my_robot)/urdf/my_robot.gazebo" />
-  <xacro:include filename="$(find my_robot)/urdf/rover_colors.gazebo" />
+<robot name="rover" xmlns:xacro="http://www.ros.org/wiki/xacro">
+  <xacro:include filename="$(find self_localizing_robot)/urdf/rover_plugins.gazebo" />
+  <xacro:include filename="$(find self_localizing_robot)/urdf/rover_colors.gazebo" />
   <link name="robot_footprint"></link>
   <joint name="robot_footprint_joint" type="fixed">
@@ -195,5 +195,5 @@
       <origin xyz="0 0 0" rpy="0 0 0"/>
       <geometry>
-	<mesh filename="package://my_robot/meshes/hokuyo.dae"/>
+	<mesh filename="package://self_localizing_robot/meshes/hokuyo.dae"/>
       </geometry>
     </visual>-->

Commit message: Add missing colors to URDF model for RVIZ

File: self_localizing_robot/urdf/rover.xacro (robot description, xacro)
@@ -31,4 +31,7 @@
         <box size=".4 .2 .1"/>
       </geometry>
+      <material name="greenish">
+        <color rgba="0.0 0.8 0.5 1.0"/>
+      </material>
     </visual>
     <collision name='back_caster_collision'>
@@ -43,4 +46,7 @@
         <sphere radius="0.05"/>
       </geometry>
+      <material name="black">
+        <color rgba="0.0 0.0 0.0 1.0"/>
+      </material>
     </visual>
     <collision name='front_caster_collision'>
@@ -55,4 +61,7 @@
         <sphere radius="0.05"/>
       </geometry>
+      <material name="black">
+        <color rgba="0.0 0.0 0.0 1.0"/>
+      </material>
     </visual>
   </link>
@@ -72,9 +81,12 @@
         <cylinder radius="0.1" length="0.05"/>
       </geometry>
+      <material name="black">
+        <color rgba="0.0 0.0 0.0 1.0"/>
+      </material>
     </visual>
     <collision>
       <origin xyz="0 0 0" rpy="0 1.5707 1.5707"/>
       <geometry>
-	 <cylinder radius="0.1" length="0.05"/>
+	      <cylinder radius="0.1" length="0.05"/>
       </geometry>
     </collision>
@@ -93,5 +105,5 @@
       <origin xyz="0 0 0" rpy="0 1.5707 1.5707"/>
       <geometry>
-	<cylinder radius="0.1" length="0.05"/>
+	      <cylinder radius="0.1" length="0.05"/>
       </geometry>
     </collision>
@@ -99,6 +111,9 @@
       <origin xyz="0 0 0" rpy="0 1.5707 1.5707"/>
       <geometry>
-	<cylinder radius="0.1" length="0.05"/>
-      </geometry>
+	      <cylinder radius="0.1" length="0.05"/>
+      </geometry>
+      <material name="black">
+        <color rgba="0.0 0.0 0.0 1.0"/>
+      </material>
     </visual>
   </link>
@@ -164,6 +179,9 @@
       <origin xyz="0 0 0" rpy="0 0 0"/>
       <geometry>
-	<box size="0.05 0.05 0.05"/>
-      </geometry>
+	       <box size="0.05 0.05 0.05"/>
+      </geometry>
+      <material name="black">
+        <color rgba="0.0 0.0 0.0 1.0"/>
+      </material>
     </visual>
     <collision>
