Commit message: feat: Add a depth camera.
Use an RGBD camera to perform graph SLAM via RTAB-Map.

File: slamming_robot/urdf/rover.xacro (robot description, xacro)
@@ -1,6 +1,6 @@
 <?xml version='1.0'?>
 <robot name="rover" xmlns:xacro="http://www.ros.org/wiki/xacro">
-  <xacro:include filename="$(find self_localizing_robot)/urdf/rover_plugins.gazebo" />
-  <xacro:include filename="$(find self_localizing_robot)/urdf/rover_colors.gazebo" />
+  <xacro:include filename="$(find slamming_robot)/urdf/rover_plugins.gazebo" />
+  <xacro:include filename="$(find slamming_robot)/urdf/rover_colors.gazebo" />
   <link name="robot_footprint"></link>
   <joint name="robot_footprint_joint" type="fixed">
@@ -200,4 +200,11 @@
       <dynamics damping="1.0" friction="1.0"/>
   </joint>
+  <link name="camera_link_optical">
+  </link>
+  <joint name="camera_optical_joint" type="fixed">
+    <origin xyz="0 0 0" rpy="-1.5707 0 -1.5707"/>
+    <parent link="camera"/>
+    <child link="camera_link_optical"/>
+  </joint>
   <link name="hokuyo">
     <inertial>

Commit message: fix: redirect to correct location of the URDF meshes

File: slamming_robot/urdf/rover.xacro (robot description, xacro)
@@ -220,5 +220,5 @@
       <origin xyz="0 0 0" rpy="0 0 0"/>
       <geometry>
-	<mesh filename="package://self_localizing_robot/meshes/hokuyo.dae"/>
+	<mesh filename="package://slamming_robot/meshes/hokuyo.dae"/>
       </geometry>
     </visual>-->
